Commit message: Replace with new robot usd and urdf.

File: assets/urdf/panda_arm.urdf (robot description, URDF)
Before this commit: robot panda_arm, 9 links, 8 joints
Links:
- added link ee_target
Joints:
- added joint ee_target_joint: type fixed, parent panda_link8, child ee_target, origin xyz=0.13 0 0.07 rpy=0 0 0
